Commit message: Initial changes for metric to USC units

File: test_models/ur/ur5.urdf (robot description, URDF)
Before this commit: robot ur5, 9 links, 8 joints
Links:
- link base_link: mass 4.0 -> 4; geometry collision mesh filename=package://ur_description/meshes/ur5/collision/base.stl scale=1 1 1; visual mesh filename=package://ur_description/meshes/ur5/visual/Base.dae scale=1 1 1
- link forearm_link: geometry collision mesh filename=package://ur_description/meshes/ur5/collision/forearm.stl scale=1 1 1; visual mesh filename=package://ur_description/meshes/ur5/visual/Forearm.dae scale=1 1 1
- link shoulder_link: geometry collision mesh filename=package://ur_description/meshes/ur5/collision/shoulder.stl scale=1 1 1; visual mesh filename=package://ur_description/meshes/ur5/visual/Shoulder.dae scale=1 1 1
- link upper_arm_link: geometry collision mesh filename=package://ur_description/meshes/ur5/collision/upper_arm.stl scale=1 1 1; visual mesh filename=package://ur_description/meshes/ur5/visual/UpperArm.dae scale=1 1 1
- link wrist_1_link: geometry collision mesh filename=package://ur_description/meshes/ur5/collision/wrist_1.stl scale=1 1 1; visual mesh filename=package://ur_description/meshes/ur5/visual/Wrist1.dae scale=1 1 1
- link wrist_2_link: geometry collision mesh filename=package://ur_description/meshes/ur5/collision/wrist_2.stl scale=1 1 1; visual mesh filename=package://ur_description/meshes/ur5/visual/Wrist2.dae scale=1 1 1
- link wrist_3_link: geometry collision mesh filename=package://ur_description/meshes/ur5/collision/wrist_3.stl scale=1 1 1; visual mesh filename=package://ur_description/meshes/ur5/visual/Wrist3.dae scale=1 1 1
Joints:
- joint ee_fixed_joint: axis (none) -> 0 0 0; origin xyz=0.0 0.0823 0.0 rpy=0.0 0.0 1.570796325 -> xyz=0 0.0823 0 rpy=0 -0 1.5708
- joint elbow_joint: limit lower=-6.2831853 upper=6.2831853 effort=150.0 velocity=3.15 -> lower=-6.28319 upper=6.28319 effort=150 velocity=3.15; origin xyz=0.0 -0.1197 0.425 rpy=0.0 0.0 0.0 -> xyz=0 -0.1197 0.425 rpy=1.22465e-16 0.523599 1.22465e-16
- joint shoulder_lift_joint: limit lower=-6.2831853 upper=6.2831853 effort=150.0 velocity=3.15 -> lower=-6.28319 upper=6.28319 effort=150 velocity=3.15; origin xyz=0.0 0.13585 0.0 rpy=0.0 1.570796325 0.0 -> xyz=0 0.13585 0 rpy=3.14159 1.57079 3.14159
- joint shoulder_pan_joint: limit lower=-6.2831853 upper=6.2831853 effort=150.0 velocity=3.15 -> lower=-6.28319 upper=6.28319 effort=150 velocity=3.15; origin xyz=0.0 0.0 0.089159 rpy=0.0 0.0 0.0 -> xyz=0 0 0.089159 rpy=0 -0 0
- joint world_joint: axis (none) -> 0 0 0; origin xyz=0.0 0.0 0.0 rpy=0.0 0.0 0.0 -> xyz=0 0 0 rpy=0 -0 0
- joint wrist_1_joint: limit lower=-6.2831853 upper=6.2831853 effort=28.0 velocity=3.2 -> lower=-6.28319 upper=6.28319 effort=28 velocity=3.2; origin xyz=0.0 0.0 0.39225 rpy=0.0 1.570796325 0.0 -> xyz=0 0 0.39225 rpy=3.14159 1.57079 3.14159
- joint wrist_2_joint: limit lower=-6.2831853 upper=6.2831853 effort=28.0 velocity=3.2 -> lower=-6.28319 upper=6.28319 effort=28 velocity=3.2; origin xyz=0.0 0.093 0.0 rpy=0.0 0.0 0.0 -> xyz=0 0.093 0 rpy=0 -0 0
- joint wrist_3_joint: limit lower=-6.2831853 upper=6.2831853 effort=28.0 velocity=3.2 -> lower=-6.28319 upper=6.28319 effort=28 velocity=3.2; origin xyz=0.0 0.0 0.09465 rpy=0.0 0.0 0.0 -> xyz=0 0 0.09465 rpy=0 -0 0

Commit message: Allowed for user specification of joint origin in inches and degrees. Added option to specify joint limits and velocities using degrees. Fixed an error in origin_property that caused the model to move to the wrong quadrant.

File: test_models/ur/ur5.urdf (robot description, URDF)
Before this commit: robot ur5, 9 links, 8 joints
Joints:
- joint elbow_joint: origin xyz=0 -0.1197 0.425 rpy=1.22465e-16 0.523599 1.22465e-16 -> xyz=0 -0.1197 0.425 rpy=0 -0 0

Commit message: Removed change to ur5 model

File: test_models/ur/ur5.urdf (robot description, URDF)
Before this commit: robot ur5, 9 links, 8 joints
Links:
- link base_link: mass 4 -> 4.0; geometry collision mesh filename=package://ur_description/meshes/ur5/collision/base.stl; visual mesh filename=package://ur_description/meshes/ur5/visual/Base.dae
- link forearm_link: geometry collision mesh filename=package://ur_description/meshes/ur5/collision/forearm.stl; visual mesh filename=package://ur_description/meshes/ur5/visual/Forearm.dae
- link shoulder_link: geometry collision mesh filename=package://ur_description/meshes/ur5/collision/shoulder.stl; visual mesh filename=package://ur_description/meshes/ur5/visual/Shoulder.dae
- link upper_arm_link: geometry collision mesh filename=package://ur_description/meshes/ur5/collision/upper_arm.stl; visual mesh filename=package://ur_description/meshes/ur5/visual/UpperArm.dae
- link wrist_1_link: geometry collision mesh filename=package://ur_description/meshes/ur5/collision/wrist_1.stl; visual mesh filename=package://ur_description/meshes/ur5/visual/Wrist1.dae
- link wrist_2_link: geometry collision mesh filename=package://ur_description/meshes/ur5/collision/wrist_2.stl; visual mesh filename=package://ur_description/meshes/ur5/visual/Wrist2.dae
- link wrist_3_link: geometry collision mesh filename=package://ur_description/meshes/ur5/collision/wrist_3.stl; visual mesh filename=package://ur_description/meshes/ur5/visual/Wrist3.dae
Joints:
- joint ee_fixed_joint: axis 0 0 0 -> (none); origin xyz=0 0.0823 0 rpy=0 -0 1.5708 -> xyz=0.0 0.0823 0.0 rpy=0.0 0.0 1.570796325
- joint elbow_joint: limit lower=-6.28319 upper=6.28319 effort=150 velocity=3.15 -> lower=-6.2831853 upper=6.2831853 effort=150.0 velocity=3.15; origin xyz=0 -0.1197 0.425 rpy=0 -0 0 -> xyz=0.0 -0.1197 0.425 rpy=0.0 0.0 0.0
- joint shoulder_lift_joint: limit lower=-6.28319 upper=6.28319 effort=150 velocity=3.15 -> lower=-6.2831853 upper=6.2831853 effort=150.0 velocity=3.15; origin xyz=0 0.13585 0 rpy=3.14159 1.57079 3.14159 -> xyz=0.0 0.13585 0.0 rpy=0.0 1.570796325 0.0
- joint shoulder_pan_joint: limit lower=-6.28319 upper=6.28319 effort=150 velocity=3.15 -> lower=-6.2831853 upper=6.2831853 effort=150.0 velocity=3.15; origin xyz=0 0 0.089159 rpy=0 -0 0 -> xyz=0.0 0.0 0.089159 rpy=0.0 0.0 0.0
- joint world_joint: axis 0 0 0 -> (none); origin xyz=0 0 0 rpy=0 -0 0 -> xyz=0.0 0.0 0.0 rpy=0.0 0.0 0.0
- joint wrist_1_joint: limit lower=-6.28319 upper=6.28319 effort=28 velocity=3.2 -> lower=-6.2831853 upper=6.2831853 effort=28.0 velocity=3.2; origin xyz=0 0 0.39225 rpy=3.14159 1.57079 3.14159 -> xyz=0.0 0.0 0.39225 rpy=0.0 1.570796325 0.0
- joint wrist_2_joint: limit lower=-6.28319 upper=6.28319 effort=28 velocity=3.2 -> lower=-6.2831853 upper=6.2831853 effort=28.0 velocity=3.2; origin xyz=0 0.093 0 rpy=0 -0 0 -> xyz=0.0 0.093 0.0 rpy=0.0 0.0 0.0
- joint wrist_3_joint: limit lower=-6.28319 upper=6.28319 effort=28 velocity=3.2 -> lower=-6.2831853 upper=6.2831853 effort=28.0 velocity=3.2; origin xyz=0 0 0.09465 rpy=0 -0 0 -> xyz=0.0 0.0 0.09465 rpy=0.0 0.0 0.0
